Commit message: EFK with GPS and IMU

File: agbot/robot_bringup/urdf/robot_description.urdf (robot description, URDF)
Before this commit: robot my_robot, 5 links, 4 joints
Links:
- added link imu_link; visual box size=${imu_length} ${imu_width} ${imu_height}
Joints:
- added joint imu_joint: type fixed, parent plate_link, child imu_link, origin xyz=${base_length/2 - imu_length/2 } ${-base_width/2 + imu_width/2} ${plate_height/2 + imu_height/2} rpy=3.1415 0 0
