Commit message: simulation under construction

File: agbot/robot_bringup/urdf/robot_description.urdf.xacro (robot description, xacro)
@@ -49,5 +49,5 @@
         </geometry>
         </collision>
-        <!-- <xacro:box_inertia m="200" w="${base_width}" d="${base_length}" h="${base_height}"/> -->
+        <xacro:box_inertia m="200" w="${base_width}" d="${base_length}" h="${base_height}"/>
     </link>
    <!-- Robot Footprint -->
@@ -75,5 +75,5 @@
       </geometry>
     </collision>
-    <xacro:box_inertia m="100" w="${base_width}" d="${base_length}" h="${plate_height}"/>
+    <xacro:box_inertia m="10" w="${base_width}" d="${base_length}" h="${plate_height}"/>
   </link>
   <!-- Plate to Base joint -->
@@ -101,5 +101,5 @@
         </geometry>
       </collision>
-      <xacro:cylinder_inertia m="20" r="${wheel_radius}" h="${wheel_width}"/>
+      <xacro:cylinder_inertia m="25" r="${wheel_radius}" h="${wheel_width}"/>
     </link>
     <!-- Wheel joint -->
@@ -187,5 +187,5 @@
         </material>
         </visual>
-        <xacro:box_inertia m="1" w="${gps_width}" d="${gps_length}" h="${gps_height}"/>
+        <xacro:box_inertia m="2" w="${gps_width}" d="${gps_length}" h="${gps_height}"/>
     </link>
     <!-- GPS Joint -->
@@ -205,5 +205,5 @@
         </material>
         </visual>
-        <xacro:cylinder_inertia m="1" r="${lidar_radius}" h="${lidar_length}"/>
+        <xacro:cylinder_inertia m="0.7" r="${lidar_radius}" h="${lidar_length}"/>
     </link>
     <!-- Lidar Joint -->
@@ -223,5 +223,5 @@
         </material>
         </visual>
-        <xacro:box_inertia m="1" w="${gps_width}" d="${gps_length}" h="${gps_height}"/>
+        <xacro:box_inertia m="0.2" w="${gps_width}" d="${gps_length}" h="${gps_height}"/>
     </link>
     <!-- imu Joint -->
@@ -229,5 +229,5 @@
         <parent link="plate_link"/>
         <child link="imu_link"/>
-        <origin xyz="${base_length/2 - imu_length/2 } ${-base_width/2 + imu_width/2} ${plate_height/2 + imu_height/2}" rpy="3.1415 0 0"/>
+        <origin xyz="${base_length/2 - imu_length/2 } ${-base_width/2 + imu_width/2} ${plate_height/2 + imu_height/2}" rpy="0 0 0"/>
     </joint>
 </robot>
