Commit message: consistent frictions for gazebo are found

File: agbot/robot_simulator/urdf_sim/robot_description_gazebo.urdf.xacro (robot description, xacro)
@@ -270,11 +270,41 @@
   <gazebo reference="right_wheel_link">
     <material>Gazebo/Black</material>
-    <mu1>10000</mu1>
-    <mu2>10000</mu2>
+    <mu1>8000</mu1>
+    <mu2>8000</mu2>
   </gazebo>
   <gazebo reference="left_wheel_link">
     <material>Gazebo/Black</material>
-    <mu1>10000</mu1>
-    <mu2>10000</mu2>
+    <mu1>8000</mu1>
+    <mu2>8000</mu2>
+  </gazebo>
+    <gazebo reference="right_wheel_box_link">
+    <material>Gazebo/Black</material>
+    <mu1>0.1</mu1>
+    <mu2>0.1</mu2>
+  </gazebo>
+  <gazebo reference="left_wheel_box_link">
+    <material>Gazebo/Black</material>
+    <mu1>0.1</mu1>
+    <mu2>0.1</mu2>
+  </gazebo>
+  <gazebo reference="right_wheel_additional_r_wheel_link">
+    <material>Gazebo/Black</material>
+    <mu1>0.2</mu1>
+    <mu2>0.2</mu2>
+  </gazebo>
+  <gazebo reference="left_wheel_additional_r_wheel_link">
+    <material>Gazebo/Black</material>
+    <mu1>0.2</mu1>
+    <mu2>0.2</mu2>
+  </gazebo>
+    <gazebo reference="right_wheel_additional_f_wheel_link">
+    <material>Gazebo/Black</material>
+    <mu1>0.2</mu1>
+    <mu2>0.2</mu2>
+  </gazebo>
+  <gazebo reference="left_wheel_additional_f_wheel_link">
+    <material>Gazebo/Black</material>
+    <mu1>0.2</mu1>
+    <mu2>0.2</mu2>
   </gazebo>
   <gazebo>
