Commit message: dwb issue resolved

File: agbot/robot_description/urdf/robot_description.urdf.xacro (robot description, xacro)
@@ -240,5 +240,5 @@
       <parent link="plate_link"/>
       <child link="base_scan"/>
-      <origin xyz="${base_length/2 - lidar_radius} 0 ${plate_height/2 + lidar_length/2}" rpy="0 0 0"/>
+      <origin xyz="${base_length/2 - lidar_radius} 0 ${plate_height/2 + lidar_length/2}" rpy="0 0 3.14159"/>
   </joint>
   <!-- imu -->
@@ -258,5 +258,5 @@
       <parent link="plate_link"/>
       <child link="imu_link"/>
-      <origin xyz="${base_length/2 - imu_length/2 } ${-base_width/2 + imu_width/2} ${plate_height/2 + imu_height/2}" rpy="0 0 0"/>
+      <origin xyz="${base_length/2 - imu_length/2 -0.065} ${-base_width/2 + imu_width/2 +0.065} ${plate_height/2 + imu_height/2}" rpy="0 0 0"/>
   </joint>
   <!-- Gazebo -->

Commit message: corrected IMU and GNSS link in URDF (NOT Real World)

File: agbot/robot_description/urdf/robot_description.urdf.xacro (robot description, xacro)
@@ -2,27 +2,28 @@
 <robot name="my_robot" xmlns:xacro="http://ros.org/wiki/xacro">
   <!-- Define robot constants -->
-  <xacro:property name="base_length" value="1.50"/>
-  <xacro:property name="base_width" value="1.03"/>
-  <xacro:property name="base_height" value="0.36"/>
-  <xacro:property name="base_zoff" value="0.16"/>
-  <xacro:property name="plate_height" value="0.04"/>
-  <xacro:property name="wheel_radius" value="0.2"/>
-  <xacro:property name="wheel_width" value="0.23"/>
-  <xacro:property name="wheel_zoff" value="0.24"/>
-  <xacro:property name="wheel_box_length" value="1.25"/>
-  <xacro:property name="lidar_radius" value="0.05"/>
-  <xacro:property name="lidar_length" value="0.05"/>
-  <xacro:property name="gps_length" value="0.15"/>
-  <xacro:property name="gps_width" value="0.15"/>
-  <xacro:property name="gps_height" value="0.1"/>
-  <xacro:property name="imu_length" value="0.02"/>
-  <xacro:property name="imu_width" value="0.02"/>
-  <xacro:property name="imu_height" value="0.007"/>
+  <xacro:property name="base_length" value="1.50" />
+  <xacro:property name="base_width" value="1.03" />
+  <xacro:property name="base_height" value="0.36" />
+  <xacro:property name="base_zoff" value="0.16" />
+  <xacro:property name="plate_height" value="0.04" />
+  <xacro:property name="wheel_radius" value="0.2" />
+  <xacro:property name="wheel_width" value="0.23" />
+  <xacro:property name="wheel_zoff" value="0.24" />
+  <xacro:property name="wheel_box_length" value="1.25" />
+  <xacro:property name="lidar_radius" value="0.05" />
+  <xacro:property name="lidar_length" value="0.05" />
+  <xacro:property name="gps_length" value="0.15" />
+  <xacro:property name="gps_width" value="0.15" />
+  <xacro:property name="gps_height" value="0.1" />
+  <xacro:property name="imu_length" value="0.02" />
+  <xacro:property name="imu_width" value="0.02" />
+  <xacro:property name="imu_height" value="0.007" />
   <!-- Define some commonly used intertial properties  -->
   <xacro:macro name="box_inertia" params="m w h d">
     <inertial>
-      <origin xyz="0 0 0" rpy="${pi/2} 0 ${pi/2}"/>
-      <mass value="${m}"/>
-      <inertia ixx="${(m/12) * (h*h + d*d)}" ixy="0.0" ixz="0.0" iyy="${(m/12) * (w*w + d*d)}" iyz="0.0" izz="${(m/12) * (w*w + h*h)}"/>
+      <origin xyz="0 0 0" rpy="${pi/2} 0 ${pi/2}" />
+      <mass value="${m}" />
+      <inertia ixx="${(m/12) * (h*h + d*d)}" ixy="0.0" ixz="0.0" iyy="${(m/12) * (w*w + d*d)}"
+        iyz="0.0" izz="${(m/12) * (w*w + h*h)}" />
     </inertial>
   </xacro:macro>
@@ -30,24 +31,25 @@
     <inertial>
       <origin xyz="0 0 0" rpy="${pi/2} 0 0" />
-      <mass value="${m}"/>
-      <inertia ixx="${(m/12) * (3*r*r + h*h)}" ixy = "0" ixz = "0" iyy="${(m/12) * (3*r*r + h*h)}" iyz = "0" izz="${(m/2) * (r*r)}"/>
+      <mass value="${m}" />
+      <inertia ixx="${(m/12) * (3*r*r + h*h)}" ixy="0" ixz="0" iyy="${(m/12) * (3*r*r + h*h)}"
+        iyz="0" izz="${(m/2) * (r*r)}" />
     </inertial>
   </xacro:macro>
   <!-- Robot Base -->
   <link name="base_link">
-      <visual>
-      <geometry>
-          <box size="${base_length} ${base_width} ${base_height}"/>
+    <visual>
+      <geometry>
+        <box size="${base_length} ${base_width} ${base_height}" />
       </geometry>
       <material name="White">
-          <color rgba="1 1 1 1.0"/>
+        <color rgba="1 1 1 1.0" />
       </material>
-      </visual>
-      <collision>
-      <geometry>
-          <box size="${base_length} ${base_width} ${base_height}"/>
-      </geometry>
-      </collision>
-      <xacro:box_inertia m="200" w="${base_width}" d="${base_length}" h="${base_height}"/>
+    </visual>
+    <collision>
+      <geometry>
+        <box size="${base_length} ${base_width} ${base_height}" />
+      </geometry>
+    </collision>
+    <xacro:box_inertia m="200" w="${base_width}" d="${base_length}" h="${base_height}" />
   </link>
   <!-- Robot Footprint -->
@@ -55,7 +57,7 @@
   </link>
   <joint name="base_joint" type="fixed">
-      <parent link="base_link"/>
-      <child link="base_footprint"/>
-      <origin xyz="0.0 0.0 ${-(base_zoff)}" rpy="0 0 0"/>
+    <parent link="base_link" />
+    <child link="base_footprint" />
+    <origin xyz="0.0 0.0 ${-(base_zoff)}" rpy="0 0 0" />
   </joint>
   <!-- Robot Plate -->
@@ -63,22 +65,22 @@
     <visual>
       <geometry>
-        <box size="${base_length} ${base_width} ${plate_height}"/>
+        <box size="${base_length} ${base_width} ${plate_height}" />
       </geometry>
       <material name="Red">
-        <color rgba="1 0 0 1.0"/>
+        <color rgba="1 0 0 1.0" />
       </material>
     </visual>
     <collision>
       <geometry>
-        <box size="${base_length} ${base_width} ${plate_height}"/>
+        <box size="${base_length} ${base_width} ${plate_height}" />
       </geometry>
     </collision>
-    <xacro:box_inertia m="10" w="${base_width}" d="${base_length}" h="${plate_height}"/>
+    <xacro:box_inertia m="10" w="${base_width}" d="${base_length}" h="${plate_height}" />
   </link>
   <!-- Plate to Base joint -->
   <joint name="plate_base_joint" type="fixed">
-    <parent link="base_link"/>
-    <child link="plate_link"/>
-    <origin xyz="0 0 ${base_height/2 + plate_height/2}" rpy="0 0 0"/>
+    <parent link="base_link" />
+    <child link="plate_link" />
+    <origin xyz="0 0 ${base_height/2 + plate_height/2}" rpy="0 0 0" />
     <!-- <axis xyz="0 0 1"/>
     <limit lower="0" upper="1" effort="1000" velocity="0.1"/> -->
@@ -88,175 +90,180 @@
     <link name="${name}_link">
       <visual>
-        <origin xyz="0 0 0" rpy="${pi/2} 0 0"/>
-        <geometry>
-          <cylinder radius="${wheel_radius}" length="${wheel_width}"/>
+        <origin xyz="0 0 0" rpy="${pi/2} 0 0" />
+        <geometry>
+          <cylinder radius="${wheel_radius}" length="${wheel_width}" />
         </geometry>
         <material name="Blue">
-          <color rgba="0 0 0.5 1.0"/>
+          <color rgba="0 0 0.5 1.0" />
         </material>
       </visual>
       <collision>
-      <origin xyz="0 0 0" rpy="${pi/2} 0 0"/>
-        <geometry>
-          <cylinder radius="${wheel_radius}" length="${wheel_width}"/>
+        <origin xyz="0 0 0" rpy="${pi/2} 0 0" />
+        <geometry>
+          <cylinder radius="${wheel_radius}" length="${wheel_width}" />
         </geometry>
       </collision>
-      <xacro:cylinder_inertia m="25" r="${wheel_radius}" h="${wheel_width}"/>
+      <xacro:cylinder_inertia m="25" r="${wheel_radius}" h="${wheel_width}" />
     </link>
     <!-- Wheel joint -->
     <joint name="${name}_joint" type="continuous">
-      <parent link="base_link"/>
-      <child link="${name}_link"/>
-      <origin xyz="0 ${y} ${-wheel_zoff}" rpy="0 0 0"/>
-      <axis xyz="0 1 0"/>
+      <parent link="base_link" />
+      <child link="${name}_link" />
+      <origin xyz="0 ${y} ${-wheel_zoff}" rpy="0 0 0" />
+      <axis xyz="0 1 0" />
     </joint>
   </xacro:macro>
   <!-- Create left and right wheel -->
-  <xacro:wheel name="left_wheel" y="${base_width/2 - wheel_width/2}"/>
-  <xacro:wheel name="right_wheel" y="${-base_width/2 + wheel_width/2}"/>
+  <xacro:wheel name="left_wheel" y="${base_width/2 - wheel_width/2}" />
+  <xacro:wheel name="right_wheel" y="${-base_width/2 + wheel_width/2}" />
   <!-- Box attached to Wheel -->
   <xacro:macro name="wheel_box" params="name y">
     <link name="${name}_box_link">
       <visual>
-          <geometry>
-          <box size="${wheel_box_length} ${wheel_radius*2} ${wheel_width}"/>
-          </geometry>
-          <material name="Blue">
-              <color rgba="0 0 0.8 1.0"/>
-          </material>
+        <geometry>
+          <box size="${wheel_box_length} ${wheel_radius*2} ${wheel_width}" />
+        </geometry>
+        <material name="Blue">
+          <color rgba="0 0 0.8 1.0" />
+        </material>
       </visual>
       <collision>
         <geometry>
-          <box size="${wheel_box_length} ${wheel_radius*2} ${wheel_width}"/>
+          <box size="${wheel_box_length} ${wheel_radius*2} ${wheel_width}" />
         </geometry>
       </collision>
-      <xacro:box_inertia m="5" w="${base_width}" d="${base_length}" h="${plate_height}"/>
+      <xacro:box_inertia m="5" w="${base_width}" d="${base_length}" h="${plate_height}" />
     </link>
     <joint name="${name}_box_joint" type="fixed">
-        <parent link="base_link"/>
-        <child link="${name}_box_link"/>
-        <origin xyz="0 ${y} ${-wheel_zoff}" rpy="${pi/2} 0 0"/>
+      <parent link="base_link" />
+      <child link="${name}_box_link" />
+      <origin xyz="0 ${y} ${-wheel_zoff}" rpy="${pi/2} 0 0" />
     </joint>
   </xacro:macro>
   <!-- Create left and right wheel_boxes -->
-  <xacro:wheel_box name="left_wheel" y="${base_width/2 - wheel_width/2 + 0.001}"/>
+  <xacro:wheel_box name="left_wheel" y="${base_width/2 - wheel_width/2 + 0.001}" />
   <xacro:wheel_box name="right_wheel" y="${-base_width/2 + wheel_width/2 -0.001}" />
   <!-- Create additional front left and right wheel_box_cylinders -->
   <xacro:macro name="additional_f_wheel" params="name">
     <link name="${name}_additional_f_wheel_link">
-        <visual>
-            <geometry>
-                <cylinder radius="${wheel_radius}" length="${wheel_width}"/>
-            </geometry>
-            <material name="Blue">
-                <color rgba="0 0 0.8 1.0"/>
-            </material>
-        </visual>
-        <collision>
-          <geometry>
-            <cylinder radius="${wheel_radius}" length="${wheel_width}"/>
-          </geometry>
-        </collision>
-        <xacro:cylinder_inertia m="10" r="${wheel_radius}" h="${wheel_width}"/>
+      <visual>
+        <geometry>
+          <cylinder radius="${wheel_radius}" length="${wheel_width}" />
+        </geometry>
+        <material name="Blue">
+          <color rgba="0 0 0.8 1.0" />
+        </material>
+      </visual>
+      <collision>
+        <geometry>
+          <cylinder radius="${wheel_radius}" length="${wheel_width}" />
+        </geometry>
+      </collision>
+      <xacro:cylinder_inertia m="10" r="${wheel_radius}" h="${wheel_width}" />
     </link>
     <joint name="${name}_additional_f_wheel_joint" type="fixed">
-        <parent link="${name}_box_link"/>
-        <child link="${name}_additional_f_wheel_link"/>
-        <origin rpy="0 0 0" xyz="${wheel_box_length/2} 0 0"/>
+      <parent link="${name}_box_link" />
+      <child link="${name}_additional_f_wheel_link" />
+      <origin rpy="0 0 0" xyz="${wheel_box_length/2} 0 0" />
     </joint>
   </xacro:macro>
   <!-- Create left and right additional wheels for each box -->
-  <xacro:additional_f_wheel name="left_wheel"/>
-  <xacro:additional_f_wheel name="right_wheel"/>
+  <xacro:additional_f_wheel name="left_wheel" />
+  <xacro:additional_f_wheel name="right_wheel" />
   <!-- Create additional rear left and right wheel_box_cylinders -->
   <xacro:macro name="additional_r_wheel" params="name">
-      <link name="${name}_additional_r_wheel_link">
-          <visual>
-            <geometry>
-                <cylinder radius="${wheel_radius}" length="${wheel_width}"/>
-            </geometry>
-            <material name="Blue">
-                <color rgba="0 0 0.8 1.0"/>
-            </material>
-          </visual>
-          <collision>
-            <geometry>
-              <cylinder radius="${wheel_radius}" length="${wheel_width}"/>
-            </geometry>
-          </collision>
-          <xacro:cylinder_inertia m="10" r="${wheel_radius}" h="${wheel_width}"/>
-      </link>
-      <joint name="${name}_additional_r_wheel_joint" type="fixed">
-          <parent link="${name}_box_link"/>
-          <child link="${name}_additional_r_wheel_link"/>
-          <origin rpy="0 0 0" xyz="${-wheel_box_length/2} 0 0"/>
-      </joint>
+    <link name="${name}_additional_r_wheel_link">
+      <visual>
+        <geometry>
+          <cylinder radius="${wheel_radius}" length="${wheel_width}" />
+        </geometry>
+        <material name="Blue">
+          <color rgba="0 0 0.8 1.0" />
+        </material>
+      </visual>
+      <collision>
+        <geometry>
+          <cylinder radius="${wheel_radius}" length="${wheel_width}" />
+        </geometry>
+      </collision>
+      <xacro:cylinder_inertia m="10" r="${wheel_radius}" h="${wheel_width}" />
+    </link>
+    <joint name="${name}_additional_r_wheel_joint" type="fixed">
+      <parent link="${name}_box_link" />
+      <child link="${name}_additional_r_wheel_link" />
+      <origin rpy="0 0 0" xyz="${-wheel_box_length/2} 0 0" />
+    </joint>
   </xacro:macro>
   <!-- Create left and right additional wheels for each box -->
-  <xacro:additional_r_wheel name="left_wheel"/>
-  <xacro:additional_r_wheel name="right_wheel"/>
+  <xacro:additional_r_wheel name="left_wheel" />
+  <xacro:additional_r_wheel name="right_wheel" />
   <!-- GPS -->
   <link name="gps_link">
-      <visual>
-      <geometry>
-          <box size="${gps_length} ${gps_width} ${gps_height}"/>
+    <visual>
+      <geometry>
+        <box size="${gps_length} ${gps_width} ${gps_height}" />
       </geometry>
       <material name="Grey">
-          <color rgba="0.5 0.5 .5 1.0"/>
+        <color rgba="0.5 0.5 .5 1.0" />
       </material>
-      </visual>
-      <collision>
-        <geometry>
-          <box size="${gps_length} ${gps_width} ${gps_height}"/>
-        </geometry>
-      </collision>
-      <xacro:box_inertia m="2" w="${gps_width}" d="${gps_length}" h="${gps_height}"/>
+    </visual>
+    <collision>
+      <geometry>
+        <box size="${gps_length} ${gps_width} ${gps_height}" />
+      </geometry>
+    </collision>
+    <xacro:box_inertia m="2" w="${gps_width}" d="${gps_length}" h="${gps_height}" />
   </link>
   <!-- GPS Joint -->
   <joint name="gps_joint" type="fixed">
-      <parent link="plate_link"/>
-      <child link="gps_link"/>
-      <origin xyz="${base_length/2 - gps_length/2 } ${base_width/2 - gps_width/2} ${plate_height/2 + gps_height/2}" rpy="0 0 0"/>
+    <parent link="plate_link" />
+    <child link="gps_link" />
+    <origin
+      xyz="0 0 ${plate_height/2 + gps_height/2}"
+      rpy="0 0 0" />
   </joint>
   <!-- Lidar -->
   <link name="base_scan">
-      <visual>
-        <geometry>
-            <cylinder radius="${lidar_radius}" length="${lidar_length}"/>
-        </geometry>
-        <material name="Black">
-            <color rgba="0 0 0 1.0"/>
-        </material>
-      </visual>
-      <collision>
-          <geometry>
-            <cylinder radius="${lidar_radius}" length="${lidar_length}"/>
-          </geometry>
-      </collision>
-      <xacro:cylinder_inertia m="0.7" r="${lidar_radius}" h="${lidar_length}"/>
+    <visual>
+      <geometry>
+        <cylinder radius="${lidar_radius}" length="${lidar_length}" />
+      </geometry>
+      <material name="Black">
+        <color rgba="0 0 0 1.0" />
+      </material>
+    </visual>
+    <collision>
+      <geometry>
+        <cylinder radius="${lidar_radius}" length="${lidar_length}" />
+      </geometry>
+    </collision>
+    <xacro:cylinder_inertia m="0.7" r="${lidar_radius}" h="${lidar_length}" />
   </link>
   <!-- Lidar Joint -->
   <joint name="scan_joint" type="fixed">
-      <parent link="plate_link"/>
-      <child link="base_scan"/>
-      <origin xyz="${base_length/2 - lidar_radius} 0 ${plate_height/2 + lidar_length/2}" rpy="0 0 3.14159"/>
+    <parent link="plate_link" />
+    <child link="base_scan" />
+    <origin xyz="${base_length/2 - lidar_radius} 0 ${plate_height/2 + lidar_length/2}"
+      rpy="0 0 3.14159" />
   </joint>
   <!-- imu -->
   <link name="imu_link">
-      <visual>
-      <geometry>
-          <box size="${imu_length} ${imu_width} ${imu_height}"/>
+    <visual>
+      <geometry>
+        <box size="${imu_length} ${imu_width} ${imu_height}" />
       </geometry>
       <material name="red">
-          <color rgba="0.5 0.2 .2 1.0"/>
+        <color rgba="0.5 0.2 .2 1.0" />
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